Commit message: feat(description): cotas del ensamblado de Fusion y paredes sobresalientes

File: ros2_ws/src/caid_description/urdf/caid_bot.urdf.xacro (robot description, xacro)
@@ -23,5 +23,7 @@
   <xacro:property name="z_piso1" value="${-(esp + sep + esp)}"/>
   <xacro:property name="z_sobre_p1" value="${-(esp + sep)}"/>   <!-- cara superior del piso 1 -->
-  <xacro:property name="alto_pared" value="0.056"/>
+  <xacro:property name="alto_pared" value="${dim['paredes']['alto'] * mm}"/>
+  <xacro:property name="d_pf" value="${dim['paredes']['frontal_sobresale'] * mm}"/>
+  <xacro:property name="d_pt" value="${dim['paredes']['trasera_sobresale'] * mm}"/>
   <!-- Caja envolvente (mm) de las mallas de las paredes: salen de leer los vértices de cada STL.
        Cada STL tiene su origen en una esquina, por eso hay que desplazarlas a mano. -->
@@ -68,5 +70,5 @@
         <!-- Pared frontal (0-2-10): giro +90° sobre z, cara curva hacia adelante, al ras del borde -->
     <visual>
-      <origin xyz="${largo/2 + pf_ymin*mm} ${-(pf_xmin + pf_xmax)/2*mm} ${z_sobre_p1 - pf_zmin*mm}" rpy="0 0 ${pi/2}"/>
+      <origin xyz="${largo/2 + d_pf + pf_ymin*mm} ${-(pf_xmin + pf_xmax)/2*mm} ${z_sobre_p1 - pf_zmin*mm}" rpy="0 0 ${pi/2}"/>
       <geometry>
         <mesh filename="package://caid_description/meshes/pared_frente.stl" scale="0.001 0.001 0.001"/>
@@ -75,10 +77,10 @@
     </visual>
     <collision>
-      <origin xyz="${largo/2 - (pf_ymax - pf_ymin)*mm/2} 0 ${z_sobre_p1 + alto_pared/2}" rpy="0 0 0"/>
+      <origin xyz="${largo/2 + d_pf - (pf_ymax - pf_ymin)*mm/2} 0 ${z_sobre_p1 + alto_pared/2}" rpy="0 0 0"/>
       <geometry><box size="${(pf_ymax - pf_ymin)*mm} ${(pf_xmax - pf_xmin)*mm} ${alto_pared}"/></geometry>
     </collision>
     <!-- Pared trasera (0-2-20): giro -90° sobre z, cara curva hacia atrás -->
     <visual>
-      <origin xyz="${-largo/2 - pt_ymin*mm} ${(pt_xmin + pt_xmax)/2*mm} ${z_sobre_p1 - pt_zmin*mm}" rpy="0 0 ${-pi/2}"/>
+      <origin xyz="${-largo/2 - d_pt - pt_ymin*mm} ${(pt_xmin + pt_xmax)/2*mm} ${z_sobre_p1 - pt_zmin*mm}" rpy="0 0 ${-pi/2}"/>
       <geometry>
         <mesh filename="package://caid_description/meshes/pared_posterior.stl" scale="0.001 0.001 0.001"/>
@@ -87,5 +89,5 @@
     </visual>
     <collision>
-      <origin xyz="${-largo/2 + (pt_ymax - pt_ymin)*mm/2} 0 ${z_sobre_p1 + alto_pared/2}" rpy="0 0 0"/>
+      <origin xyz="${-largo/2 - d_pt + (pt_ymax - pt_ymin)*mm/2} 0 ${z_sobre_p1 + alto_pared/2}" rpy="0 0 0"/>
       <geometry><box size="${(pt_ymax - pt_ymin)*mm} ${(pt_xmax - pt_xmin)*mm} ${alto_pared}"/></geometry>
     </collision>

Commit message: feat(description): sensores, cámara con giro y piezas modificadas del ensamblado

File: ros2_ws/src/caid_description/urdf/caid_bot.urdf.xacro (robot description, xacro)
@@ -37,4 +37,5 @@
   <material name="pla_hueso"><color rgba="0.93 0.91 0.82 1.0"/></material>
   <material name="goma"><color rgba="0.05 0.05 0.05 1.0"/></material>
+  <material name="pla_negro"><color rgba="0.12 0.12 0.12 1.0"/></material>
   <link name="base_footprint"/>
   <joint name="base_footprint_joint" type="fixed">
@@ -46,5 +47,5 @@
     <!-- Piso 2 (arriba) -->
     <visual>
-      <origin xyz="0 0 ${z_piso2}" rpy="0 0 0"/>
+      <origin xyz="0 0 ${z_piso2}" rpy="0 0 ${pi}"/>
       <geometry>
         <mesh filename="package://caid_description/meshes/chasis_armadillo.stl" scale="0.001 0.001 0.001"/>
@@ -58,7 +59,7 @@
     <!-- Piso 1 (abajo) -->
     <visual>
-      <origin xyz="0 0 ${z_piso1}" rpy="0 0 0"/>
+      <origin xyz="0 0 ${z_piso1}" rpy="0 0 ${pi}"/>
       <geometry>
-        <mesh filename="package://caid_description/meshes/chasis_armadillo.stl" scale="0.001 0.001 0.001"/>
+        <mesh filename="package://caid_description/meshes/chasis_armadillo_inferior.stl" scale="0.001 0.001 0.001"/>
       </geometry>
       <material name="acrilico"/>
@@ -82,5 +83,5 @@
     <!-- Pared trasera (0-2-20): giro -90° sobre z, cara curva hacia atrás -->
     <visual>
-      <origin xyz="${-largo/2 - d_pt - pt_ymin*mm} ${(pt_xmin + pt_xmax)/2*mm} ${z_sobre_p1 - pt_zmin*mm}" rpy="0 0 ${-pi/2}"/>
+      <origin xyz="0 0 ${z_piso1}" rpy="0 0 ${pi}"/>
       <geometry>
         <mesh filename="package://caid_description/meshes/pared_posterior.stl" scale="0.001 0.001 0.001"/>
@@ -119,3 +120,53 @@
   <xacro:rueda name="wheel_rl" x="${x_tras}" y="${y_rueda}"/>
   <xacro:rueda name="wheel_rr" x="${x_tras}" y="${-y_rueda}"/>
+  <!-- ===== Ultrasonidos: un marco por sensor, en el punto medio entre sus dos ojos ===== -->
+  <xacro:property name="us_f" value="${dim['sensores_ultrasonido']['frontal']}"/>
+  <xacro:property name="us_l" value="${dim['sensores_ultrasonido']['lateral_izquierdo']}"/>
+  <xacro:property name="us_r" value="${dim['sensores_ultrasonido']['lateral_derecho']}"/>
+  <!-- El eje x del marco apunta hacia donde mira el sensor; yaw gira ese eje sobre z. -->
+  <xacro:macro name="ultrasonido" params="name x y z yaw">
+    <link name="${name}"/>
+    <joint name="${name}_joint" type="fixed">
+      <parent link="base_link"/>
+      <child link="${name}"/>
+      <origin xyz="${x} ${y} ${z}" rpy="0 0 ${yaw}"/>
+    </joint>
+  </xacro:macro>
+  <xacro:ultrasonido name="us_front" x="${us_f['x']*mm}" y="${us_f['y']*mm}" z="${us_f['z']*mm}" yaw="0"/>
+  <xacro:ultrasonido name="us_left"  x="${us_l['x']*mm}" y="${us_l['y']*mm}" z="${us_l['z']*mm}" yaw="${pi/2}"/>
+  <xacro:ultrasonido name="us_right" x="${us_r['x']*mm}" y="${us_r['y']*mm}" z="${us_r['z']*mm}" yaw="${-pi/2}"/>
+  <!-- ===== Cámara: giro (revolute) -> cuerpo -> marco óptico (REP-103) ===== -->
+  <xacro:property name="cam" value="${dim['camara']}"/>
+  <xacro:property name="cam_x" value="0.0141"/>   <!-- espesor de la caja, del ensamblado -->
+  <xacro:property name="cam_y" value="0.0352"/>
+  <xacro:property name="cam_z" value="0.0447"/>
+  <link name="camera_pan_link">
+    <xacro:box_inertia m="0.01" x="0.03" y="0.03" z="0.02"/>
+  </link>
+  <joint name="camera_pan_joint" type="revolute">
+    <parent link="base_link"/>
+    <child link="camera_pan_link"/>
+    <origin xyz="${cam['x']*mm} ${cam['y']*mm} 0" rpy="0 0 0"/>
+    <axis xyz="0 0 1"/>
+    <limit lower="${-pi/2}" upper="${pi/2}" effort="0.2" velocity="3.0"/>
+  </joint>
+  <link name="camera_link">
+    <visual>
+      <origin xyz="0 0 0" rpy="0 0 0"/>
+      <geometry><box size="${cam_x} ${cam_y} ${cam_z}"/></geometry>
+      <material name="pla_negro"/>
+    </visual>
+    <xacro:box_inertia m="0.02" x="${cam_x}" y="${cam_y}" z="${cam_z}"/>
+  </link>
+  <joint name="camera_joint" type="fixed">
+    <parent link="camera_pan_link"/>
+    <child link="camera_link"/>
+    <origin xyz="0 0 ${cam['z']*mm}" rpy="0 0 0"/>
+  </joint>
+  <link name="camera_optical_frame"/>
+  <joint name="camera_optical_joint" type="fixed">
+    <parent link="camera_link"/>
+    <child link="camera_optical_frame"/>
+    <origin xyz="${cam_x/2} 0 0" rpy="${-pi/2} 0 ${-pi/2}"/>
+  </joint>
 </robot>
